Commit message: fix namespace in simulation

File: kobuki_description/urdf/kobuki_gazebo.urdf.xacro (robot description, xacro)
@@ -1,5 +1,7 @@
 <?xml version="1.0"?>
 <robot name="kobuki_sim" xmlns:xacro="http://ros.org/wiki/xacro">
-  <xacro:macro name="kobuki_sim">
+	<xacro:arg name="namespace" default=""/>
+	<xacro:property name="robot_namespace" value="/$(arg namespace)"/>
+  	<xacro:macro name="kobuki_sim">
 	  <gazebo reference="wheel_left_link">
 	    <mu1>1.0</mu1>
@@ -171,4 +173,9 @@
       <plugin name="differential_drive_controller" filename="libgazebo_ros_diff_drive.so">
         <update_rate>10</update_rate>
+		<ros>
+		    <namespace>${robot_namespace}</namespace>
+			<remapping>/tf:=tf</remapping>
+			<remapping>/tf_static:=tf_static</remapping>
+        </ros>
         <left_joint>wheel_left_joint</left_joint>
         <right_joint>wheel_right_joint</right_joint>
